Commit message: Update stella.xacro

File: stella_description/urdf/stella.xacro (robot description, xacro)
@@ -28,5 +28,5 @@
     </collision>
     <inertial>
-      <origin xyz="0 0 0" rpy="0 0 0"/>
+      <origin xyz="0 0 ${bodyHeight/2}" rpy="0 0 0"/>
       <mass value="${bodyMass}"/>
       <inertia ixx="${bodyMass*(bodyLength*bodyLength+bodyHeight*bodyHeight)/12}" ixy="0" ixz="0"

Commit message: Update stella.xacro

File: stella_description/urdf/stella.xacro (robot description, xacro)
@@ -44,5 +44,5 @@
     <parent link="base_link"/>
     <child link="base_scan"/>
-    <origin xyz="${bodyLength/2 - 0.075} 0 0.229" rpy="0 0 ${PI}"/>
+    <origin xyz="${bodyLength/2 - 0.075} 0 0.248" rpy="0 0 ${PI}"/>
   </joint>
   <link name="base_scan" />
